File: 2016.07.18_BatteryPoweredGenericV2.kicad_pcb (KiCad board)
At the start: 2 copper layers, 22 parts, among them P1 CONN_01X02, P2 USB_B, P3 CONN_01X03, P4 CONN_01X07, P5 CONN_01X14, P6 CONN_01X04, P7 CONN_01X03, SW1 SW_PUSH, SW2 SW_PUSH, U1 HT7333-SOT-89, U2 ESP-12E

Commit message: Version 2.0
Connections:
- P5 pad 11: /GPIO14 -> /GPIO16
- P5 pad 14: /GPIO16 -> /GPIO14
- R9 pad 1: /GPIO14 -> /GPIO16
- R9 pad 2: /GPIO14 -> /GPIO16
Routing:
- net +3V3: track 195.2 -> 208.6 mm
- net /GPIO14: track 51.2 -> 58.3 mm
- net /GPIO16: track 56.0 -> 58.8 mm
Other:
- net class 12V added: clearance 0.18, trace_width 0.6, via_dia 0.6, via_drill 0.4
- board text added: "JG Rev.2 2016.09.01"
- board text removed: "JG Rev.1 2016.07.04"
