File: 2016.07.18_BatteryPoweredGenericV2.sch (KiCad schematic (older format))
At the start: 22 parts, among them P1 CONN_01X02, P2 USB_B, P3 CONN_01X03, P4 CONN_01X07, P5 CONN_01X14, P6 CONN_01X04, P7 CONN_01X03, SW1 SW_PUSH, SW2 SW_PUSH, U1 HT7333-SOT-89, U2 ESP-12E

Commit message: Version 2.0
Changed lines of the file:
@@
 LIBS:lm1117
 LIBS:lm1117-SMD
-LIBS:2016.07.18_BatteryPoweredGeneric-cache
+LIBS:2016.07.18_BatteryPoweredGenericV2-cache
 EELAYER 25 0
 EELAYER END
@@
 SCLK
 Text Label 8950 2400 0    60   ~ 0
-GPIO14
+GPIO16
 Text Label 8950 3200 0    60   ~ 0
 GPIO13
@@
 SCLK
 Text Label 8950 2100 0    60   ~ 0
-GPIO16
+GPIO14
 Text Label 9050 4650 0    60   ~ 0
 GPIO10
@@
 Connection ~ 2550 6200
 Text Label 2550 6200 3    60   ~ 0
-GPIO14
+GPIO16
 Wire Wire Line
 	2550 6200 2550 6450
